File: hardware/poopvolt.kicad_sch (KiCad schematic)
At the start: 10 parts, among them J1 I2C port / AHT20, J2 I2C port / LCD, J3 UART port / PN532, J4 A0 port / light, P1 Laptop USB-C supply, U1 UNO Q + Base Shield, U2 Grove AHT20 / 0x38, U3 Grove LCD 16x2 / 0x3E, U4 Grove PN532 / HSU, U5 Grove Light Sensor (P)

Commit message: docs(hardware): add solar path to KiCad schematic; replication guide
Schematic: Grove A1 port + 2.5A current sensor (PV_ISENSE_A1), and the
separate solar path panel -> current sensor -> Waveshare Solar Power
Manager -> LiPo. ERC clean, 15-net connectivity check passes (A3 sheet).
Guide: step-by-step rebuild on Ubuntu 24.04 with current status.

Co-Authored-By: Claude Opus 5.5 <noreply@anthropic.com>
Parts:
- added BT1: LiPo 3.7 V 1000 mAh, symbol PoopVolt:LiPo_1S
- added J5: A1 port / PV current, symbol PoopVolt:Grove_A1
- added PV1: Mini solar panel R1123, symbol PoopVolt:Solar_Panel
- added U6: Grove 2.5A DC current (ACS70331), symbol PoopVolt:Current_Sensor_2A5
- added U7: Waveshare Solar Power Manager (5 V / 1 A), symbol PoopVolt:Solar_Power_Manager
Connections:
- net +3V3: now also J5.3 (VCC), U6.3 (VCC)
- net GND: now also J5.4 (GND), U6.4 (GND)
- net SPARE_A1 renamed PV_ISENSE_A1
- net PV_ISENSE_A1: now also J5.1 (A1), U6.1 (OUT)
- new net BAT_NEG: BT1.NEG (-), U7.BAT- (BAT-(PH2.0))
- new net BAT_POS: BT1.POS (+), U7.BAT+ (BAT+(PH2.0))
- new net PV_NEG: PV1.NEG (-), U7.SOL- (SOLAR_IN-)
- new net PV_POS: PV1.POS (+), U6.IP+ (IN+)
- new net PV_TO_CHARGER: U6.IP- (IN-), U7.SOL+ (SOLAR_IN+)
- new net SPARE_A2: J5.2 (A2), U1.A2 (PA6 / spare), U6.2 (NC / unused)
Other:
- note added: "800 mV/A zero 266.5 mV"
- note added: "90 x 60 mm rating unverified"
- note added: "As built in PR #49 - 10 October 2026 - UNO Q on USB power, 3.3 V Grove ports, solar panel charges a LiPo through the Waveshare manager"
- note added: "CN3791 MPPT charger MPPT SET = 6 V Battery switch ON USB OUT not connected"
- note added: "Current sensor U6 is in series on the panel + wire: PV_POS -> IN+ ... IN- -> PV_TO_CHARGER -> SOLAR IN +. The solar side shares no conductor with the UNO Q or Grove GND."
- note added: "Disconnected: Modulino Movement, Media Carrier, Waveshare USB OUT (5 V / 1 A). Rejected: HRS1358 + LM2596 step-down feeding the UNO Q (a buck cannot make 5 V from a 3.7 V LiPo). Wi-Fi phone camera integration remains outside this wiring."
- note added: "Pin 2: unused A1 carries PV current"
- note added: "SOLAR HARVESTING (separate from the UNO Q supply)"
- note removed: "As built in PR #49 - 10 October 2026 - USB power, 3.3 V Grove ports"
- note removed: "Disconnected: ACS70331 current sensor, Modulino Movement, Media Carrier. Solar / battery / converter power and Wi-Fi camera integration remain outside this wiring."
- note removed: "Pin 2: unused A1 not sampled"
